File: _autosave-audio-switch.sch (KiCad schematic (older format))
At the start: 17 parts, among them J1 OUT_1, U1 Pico, U2 CD4052B, U3 CD4052B

Commit message: Remove pico and use sr latch for input slection
Parts:
- removed U1: Pico, pi:RPi_Pico_SMD_TH, symbol MCU_RaspberryPi_and_Boards:Pico
- added D5, D6, D7, D8: D_Small, Diode_SMD:D_0805_2012Metric_Pad1.15x1.40mm_HandSolder, symbol Device:D_Small
- added R1, R2, R3, R4: R_Small, Resistor_SMD:R_0805_2012Metric_Pad1.20x1.40mm_HandSolder, symbol Device:R_Small
- added U4: 7402, Package_DIP:DIP-14_W7.62mm, symbol 74xx:7402
- MX1, MX2, MX3, MX4: footprint (none) -> MX_Only:MXOnly-1U
- OUT_2: value AudioJack4_Out -> OUT_2
- U2, U3: footprint Package_DIP:DIP-16_W7.62mm_Socket -> Package_DIP:DIP-16_W7.62mm
- renumbered IN_1 to IN_0, IN_4 to IN_1, J1 to OUT_1
Connections:
- net labels added: Select_A_HIGH, Select_A_LOW, Select_B_HIGH, Select_B_LOW
- net labels removed: +3.3V, Col0, Col1, GNDA, I2S_bck, I2S_data, I2S_lrck, Row0, Row1, mute
- wire segments 139 -> 132
Other:
- moved on the sheet: IN_0, IN_1, IN_2, IN_3, OUT_1, OUT_2, U2, U3
