File: Amp.sch (KiCad schematic (older format))
At the start: 30 parts, among them U501 LM386

Commit message: Latch
Parts:
- removed BASS401, Bass?, GAIN401, Gain?, VOL401, Volume?: 10k, Potentiometer_THT:Potentiometer_Alps_RK09L_Double_Vertical, symbol Device:R_POT_Dual_Separate
- added BASS301, GAIN301, VOL301: 10k, Potentiometer_THT:Potentiometer_Alps_RK09L_Double_Vertical, symbol Device:R_POT_Dual_Separate
- gave numbers to parts that had none: 12
Connections:
- net GND: now also VOL301.3, VOL301.6
- net Input_Left: now also VOL301.4
- net Input_Right: now also VOL301.1
- net at U401.3 (+): now also VOL301.2
- net at U401.1 (GAIN): now also BASS301.2, GAIN301.2
- net at C407.1: now also BASS301.3
- net at C405.1: now also GAIN301.3
- net at U501.3 (+): now also VOL301.5
- net at U501.1 (GAIN): now also BASS301.5, GAIN301.5
- net at C507.1: now also BASS301.6
- net at C505.1: now also GAIN301.6
