File: Amp.sch (KiCad schematic (older format))
At the start: 27 parts, among them U401 LM386, U402 LM386

Commit message: Test
Parts:
- BASS401, GAIN401, VOL401: footprint (none) -> audio-switch:dual_pot_jaycar
- C401, C403, C404, C407, C408, C410, C412, C413, C416, C417: footprint (none) -> Capacitor_SMD:C_0805_2012Metric_Pad1.18x1.45mm_HandSolder
- C402, C405, C406, C411, C414, C415: footprint (none) -> Capacitor_Tantalum_SMD:CP_EIA-2012-15_AVX-P_Pad1.30x1.05mm_HandSolder
- C409, C418: footprint (none) -> Capacitor_THT:CP_Radial_D12.5mm_P5.00mm
- R401, R402, R403, R404: footprint (none) -> Resistor_SMD:R_0805_2012Metric_Pad1.20x1.40mm_HandSolder
Changed lines of the file:
@@
 F 0 "GAIN401" H 8031 4446 50  0000 R CNN
 F 1 "10kΩ" H 8031 4355 50  0000 R CNN
-F 2 "" H 8100 4400 50  0001 C CNN
+F 2 "audio-switch:dual_pot_jaycar" H 8100 4400 50  0001 C CNN
 F 3 "~" H 8100 4400 50  0001 C CNN
 	2    8100 4400
@@
 F 0 "GAIN401" H 4180 4396 50  0000 R CNN
 F 1 "10kΩ" H 4180 4305 50  0000 R CNN
-F 2 "" H 4250 4350 50  0001 C CNN
+F 2 "audio-switch:dual_pot_jaycar" H 4250 4350 50  0001 C CNN
 F 3 "~" H 4250 4350 50  0001 C CNN
 	1    4250 4350
@@
 F 0 "BASS401" H 8480 4704 50  0000 R CNN
 F 1 "10kΩ" H 8480 4795 50  0000 R CNN
-F 2 "" H 8550 4750 50  0001 C CNN
+F 2 "audio-switch:dual_pot_jaycar" H 8550 4750 50  0001 C CNN
 F 3 "~" H 8550 4750 50  0001 C CNN
 	2    8550 4750
@@
 F 0 "BASS401" H 4630 4654 50  0000 R CNN
 F 1 "10kΩ" H 4630 4745 50  0000 R CNN
-F 2 "" H 4700 4700 50  0001 C CNN
+F 2 "audio-switch:dual_pot_jaycar" H 4700 4700 50  0001 C CNN
 F 3 "~" H 4700 4700 50  0001 C CNN
 	1    4700 4700
@@
 F 0 "VOL401" H 6980 3446 50  0000 R CNN
 F 1 "10kΩ" H 6980 3355 50  0000 R CNN
-F 2 "" H 7050 3400 50  0001 C CNN
+F 2 "audio-switch:dual_pot_jaycar" H 7050 3400 50  0001 C CNN
 F 3 "~" H 7050 3400 50  0001 C CNN
 	2    7050 3400
@@
 F 0 "VOL401" H 3131 3396 50  0000 R CNN
 F 1 "10kΩ" H 3131 3305 50  0000 R CNN
-F 2 "" H 3200 3350 50  0001 C CNN
+F 2 "audio-switch:dual_pot_jaycar" H 3200 3350 50  0001 C CNN
 F 3 "~" H 3200 3350 50  0001 C CNN
 	1    3200 3350
@@
 F 0 "C418" V 8995 3750 50  0000 C CNN
 F 1 "1000µF" V 9086 3750 50  0000 C CNN
-F 2 "" H 9288 3600 50  0001 C CNN
+F 2 "Capacitor_THT:CP_Radial_D12.5mm_P5.00mm" H 9288 3600 50  0001 C CNN
 F 3 "~" H 9250 3750 50  0001 C CNN
 	1    9250 3750
@@
 F 0 "R403" V 8357 3050 50  0000 C CNN
 F 1 "10kΩ" V 8266 3050 50  0000 C CNN
-F 2 "" V 8080 3050 50  0001 C CNN
+F 2 "Resistor_SMD:R_0805_2012Metric_Pad1.20x1.40mm_HandSolder" V 8080 3050 50  0001 C CNN
 F 3 "~" H 8150 3050 50  0001 C CNN
 	1    8150 3050
@@
 F 0 "C415" V 8805 3050 50  0000 C CNN
 F 1 "10µF" V 8714 3050 50  0000 C CNN
-F 2 "" H 8588 2900 50  0001 C CNN
+F 2 "Capacitor_Tantalum_SMD:CP_EIA-2012-15_AVX-P_Pad1.30x1.05mm_HandSolder" H 8588 2900 50  0001 C CNN
 F 3 "~" H 8550 3050 50  0001 C CNN
 	1    8550 3050
@@
 F 0 "C413" V 7750 3950 50  0000 C CNN
 F 1 "470pF" V 7850 3950 50  0000 C CNN
-F 2 "" H 7650 3950 50  0001 C CNN
+F 2 "Capacitor_SMD:C_0805_2012Metric_Pad1.18x1.45mm_HandSolder" H 7650 3950 50  0001 C CNN
 F 3 "~" H 7650 3950 50  0001 C CNN
 	1    7650 3950
@@
 F 0 "C412" V 7779 2750 50  0000 C CNN
 F 1 "0.1µF" V 7688 2750 50  0000 C CNN
-F 2 "" H 7550 2750 50  0001 C CNN
+F 2 "Capacitor_SMD:C_0805_2012Metric_Pad1.18x1.45mm_HandSolder" H 7550 2750 50  0001 C CNN
 F 3 "~" H 7550 2750 50  0001 C CNN
 	1    7550 2750
@@
 F 0 "C411" V 7295 2350 50  0000 C CNN
 F 1 "100µF" V 7386 2350 50  0000 C CNN
-F 2 "" H 7588 2200 50  0001 C CNN
+F 2 "Capacitor_Tantalum_SMD:CP_EIA-2012-15_AVX-P_Pad1.30x1.05mm_HandSolder" H 7588 2200 50  0001 C CNN
 F 3 "~" H 7550 2350 50  0001 C CNN
 	1    7550 2350
@@
 F 0 "C410" H 7392 3246 50  0000 L CNN
 F 1 "0.1µF" H 7392 3155 50  0000 L CNN
-F 2 "" H 7300 3200 50  0001 C CNN
+F 2 "Capacitor_SMD:C_0805_2012Metric_Pad1.18x1.45mm_HandSolder" H 7300 3200 50  0001 C CNN
 F 3 "~" H 7300 3200 50  0001 C CNN
 	1    7300 3200
@@
 F 0 "C417" H 8842 3696 50  0000 L CNN
 F 1 "0.1µF" H 8842 3605 50  0000 L CNN
-F 2 "" H 8750 3650 50  0001 C CNN
+F 2 "Capacitor_SMD:C_0805_2012Metric_Pad1.18x1.45mm_HandSolder" H 8750 3650 50  0001 C CNN
 F 3 "~" H 8750 3650 50  0001 C CNN
 	1    8750 3650
@@
 F 0 "R404" H 8820 3996 50  0000 L CNN
 F 1 "10Ω" H 8820 3905 50  0000 L CNN
-F 2 "" V 8680 3950 50  0001 C CNN
+F 2 "Resistor_SMD:R_0805_2012Metric_Pad1.20x1.40mm_HandSolder" V 8680 3950 50  0001 C CNN
 F 3 "~" H 8750 3950 50  0001 C CNN
 	1    8750 3950
@@
 F 0 "C416" H 8642 3696 50  0000 L CNN
 F 1 "0.033µF" H 8642 3605 50  0000 L CNN
-F 2 "" H 8550 3650 50  0001 C CNN
+F 2 "Capacitor_SMD:C_0805_2012Metric_Pad1.18x1.45mm_HandSolder" H 8550 3650 50  0001 C CNN
 F 3 "~" H 8550 3650 50  0001 C CNN
 	1    8550 3650
@@
 F 0 "C414" H 7982 4004 50  0000 R CNN
 F 1 " 10µF" H 7982 4095 50  0000 R CNN
-F 2 "" H 8138 3900 50  0001 C CNN
+F 2 "Capacitor_Tantalum_SMD:CP_EIA-2012-15_AVX-P_Pad1.30x1.05mm_HandSolder" H 8138 3900 50  0001 C CNN
 F 3 "~" H 8100 4050 50  0001 C CNN
 	1    8100 4050
@@
 F 0 "C409" V 5145 3700 50  0000 C CNN
 F 1 "1000µF" V 5236 3700 50  0000 C CNN
-F 2 "" H 5438 3550 50  0001 C CNN
+F 2 "Capacitor_THT:CP_Radial_D12.5mm_P5.00mm" H 5438 3550 50  0001 C CNN
 F 3 "~" H 5400 3700 50  0001 C CNN
 	1    5400 3700
@@
 F 0 "R401" V 4507 3000 50  0000 C CNN
 F 1 "10kΩ" V 4416 3000 50  0000 C CNN
-F 2 "" V 4230 3000 50  0001 C CNN
+F 2 "Resistor_SMD:R_0805_2012Metric_Pad1.20x1.40mm_HandSolder" V 4230 3000 50  0001 C CNN
 F 3 "~" H 4300 3000 50  0001 C CNN
 	1    4300 3000
@@
 F 0 "C406" V 4955 3000 50  0000 C CNN
 F 1 "10µF" V 4864 3000 50  0000 C CNN
-F 2 "" H 4738 2850 50  0001 C CNN
+F 2 "Capacitor_Tantalum_SMD:CP_EIA-2012-15_AVX-P_Pad1.30x1.05mm_HandSolder" H 4738 2850 50  0001 C CNN
 F 3 "~" H 4700 3000 50  0001 C CNN
 	1    4700 3000
@@
 F 0 "C404" V 3900 3900 50  0000 C CNN
 F 1 "470pF" V 4000 3900 50  0000 C CNN
-F 2 "" H 3800 3900 50  0001 C CNN
+F 2 "Capacitor_SMD:C_0805_2012Metric_Pad1.18x1.45mm_HandSolder" H 3800 3900 50  0001 C CNN
 F 3 "~" H 3800 3900 50  0001 C CNN
 	1    3800 3900
@@
 F 0 "C403" V 3929 2700 50  0000 C CNN
 F 1 "0.1µF" V 3838 2700 50  0000 C CNN
-F 2 "" H 3700 2700 50  0001 C CNN
+F 2 "Capacitor_SMD:C_0805_2012Metric_Pad1.18x1.45mm_HandSolder" H 3700 2700 50  0001 C CNN
 F 3 "~" H 3700 2700 50  0001 C CNN
 	1    3700 2700
@@
 F 0 "C402" V 3445 2300 50  0000 C CNN
 F 1 "100µF" V 3536 2300 50  0000 C CNN
-F 2 "" H 3738 2150 50  0001 C CNN
+F 2 "Capacitor_Tantalum_SMD:CP_EIA-2012-15_AVX-P_Pad1.30x1.05mm_HandSolder" H 3738 2150 50  0001 C CNN
 F 3 "~" H 3700 2300 50  0001 C CNN
 	1    3700 2300
 	0    1    1    0
 $EndComp
-Wire Wire Line
-	3850 2300 3950 2300
-Wire Wire Line
-	3950 2300 3950 2700
-Wire Wire Line
-	3950 2700 3800 2700
 $Comp
 L power:GND #PWR?
@@
 F 0 "C401" H 3542 3196 50  0000 L CNN
 F 1 "0.1µF" H 3542 3105 50  0000 L CNN
-F 2 "" H 3450 3150 50  0001 C CNN
+F 2 "Capacitor_SMD:C_0805_2012Metric_Pad1.18x1.45mm_HandSolder" H 3450 3150 50  0001 C CNN
 F 3 "~" H 3450 3150 50  0001 C CNN
 	1    3450 3150
 	1    0    0    -1
 $EndComp
-Wire Wire Line
-	3450 3050 3950 3050
 Wire Wire Line
 	3450 3750 3950 3750
@@
 F 0 "C408" H 4992 3646 50  0000 L CNN
 F 1 "0.1µF" H 4992 3555 50  0000 L CNN
-F 2 "" H 4900 3600 50  0001 C CNN
+F 2 "Capacitor_SMD:C_0805_2012Metric_Pad1.18x1.45mm_HandSolder" H 4900 3600 50  0001 C CNN
 F 3 "~" H 4900 3600 50  0001 C CNN
 	1    4900 3600
@@
 F 0 "R402" H 4970 3946 50  0000 L CNN
 F 1 "10Ω" H 4970 3855 50  0000 L CNN
-F 2 "" V 4830 3900 50  0001 C CNN
+F 2 "Resistor_SMD:R_0805_2012Metric_Pad1.20x1.40mm_HandSolder" V 4830 3900 50  0001 C CNN
 F 3 "~" H 4900 3900 50  0001 C CNN
 	1    4900 3900
@@
 F 0 "C407" H 4792 3646 50  0000 L CNN
 F 1 "0.033µF" H 4792 3555 50  0000 L CNN
-F 2 "" H 4700 3600 50  0001 C CNN
+F 2 "Capacitor_SMD:C_0805_2012Metric_Pad1.18x1.45mm_HandSolder" H 4700 3600 50  0001 C CNN
 F 3 "~" H 4700 3600 50  0001 C CNN
 	1    4700 3600
@@
 Wire Wire Line
 	3450 3250 3450 3750
-Wire Wire Line
-	3950 3050 3950 2700
-Connection ~ 3950 2700
 Wire Wire Line
 	3350 3350 3750 3350
@@
 F 0 "C405" H 4132 3954 50  0000 R CNN
 F 1 " 10µF" H 4132 4045 50  0000 R CNN
-F 2 "" H 4288 3850 50  0001 C CNN
+F 2 "Capacitor_Tantalum_SMD:CP_EIA-2012-15_AVX-P_Pad1.30x1.05mm_HandSolder" H 4288 3850 50  0001 C CNN
 F 3 "~" H 4250 4000 50  0001 C CNN
 	1    4250 4000
@@
 Wire Wire Line
 	4150 3800 4250 3800
-Wire Wire Line
-	3950 3150 3950 3050
-Connection ~ 3950 3050
 Wire Wire Line
 	3450 2800 3450 2700
@@
 Connection ~ 7800 2350
 Wire Wire Line
+	7900 4750 8400 4750
+Wire Wire Line
+	4050 4700 4550 4700
+Wire Wire Line
+	8100 4550 8100 4650
+Wire Wire Line
+	8550 5000 8550 4900
+Wire Wire Line
+	8550 3750 8550 4600
+Wire Wire Line
+	7900 4400 7900 4750
+Wire Wire Line
+	4050 4350 4050 4700
+Wire Wire Line
+	4700 3700 4700 4550
+Wire Wire Line
+	4700 4950 4700 4850
+Wire Wire Line
+	4250 4600 4250 4500
+Wire Wire Line
 	3950 2000 3950 2300
+Wire Wire Line
+	3450 3050 3950 3050
+Connection ~ 3950 3050
+Wire Wire Line
+	3950 3050 3950 3150
+Wire Wire Line
+	3800 2700 3950 2700
+Connection ~ 3950 2700
+Wire Wire Line
+	3950 2700 3950 3050
+Wire Wire Line
+	3850 2300 3950 2300
 Connection ~ 3950 2300
 Wire Wire Line
-	7900 4750 8400 4750
-Wire Wire Line
-	4050 4700 4550 4700
-Wire Wire Line
-	8100 4550 8100 4650
-Wire Wire Line
-	8550 5000 8550 4900
-Wire Wire Line
-	8550 3750 8550 4600
-Wire Wire Line
-	7900 4400 7900 4750
-Wire Wire Line
-	4050 4350 4050 4700
-Wire Wire Line
-	4700 3700 4700 4550
-Wire Wire Line
-	4700 4950 4700 4850
-Wire Wire Line
-	4250 4600 4250 4500
+	3950 2300 3950 2700
 $EndSCHEMATC
