File: Right_Amp.sch (KiCad schematic (older format))
At the start: 14 parts, among them U401 LM386

Commit message: Latch
Parts:
- removed C401, C403, C408: 0.1u, Capacitor_SMD:C_0805_2012Metric_Pad1.18x1.45mm_HandSolder, symbol Device:C_Small
- removed C402: 100u, Capacitor_SMD:C_0805_2012Metric_Pad1.18x1.45mm_HandSolder, symbol Device:CP
- removed C404: 470p, Capacitor_SMD:C_0805_2012Metric_Pad1.18x1.45mm_HandSolder, symbol Device:C_Small
- removed C405, C406: 10u, Capacitor_SMD:C_0805_2012Metric_Pad1.18x1.45mm_HandSolder, symbol Device:CP
- removed C407: 0.033u, Capacitor_SMD:C_0805_2012Metric_Pad1.18x1.45mm_HandSolder, symbol Device:C_Small
- removed C409: 1000u, Capacitor_SMD:C_0805_2012Metric_Pad1.18x1.45mm_HandSolder, symbol Device:CP
- removed R401: 10k, Resistor_SMD:R_0805_2012Metric_Pad1.20x1.40mm_HandSolder, symbol Device:R
- removed R402: 10, Resistor_SMD:R_0805_2012Metric_Pad1.20x1.40mm_HandSolder, symbol Device:R
- removed RV401, RV402: 10k, Potentiometer_THT:Potentiometer_Vishay_148-149_Dual_Horizontal, symbol Device:R_POT_Dual_Separate
- removed U401: LM386, Package_DIP:DIP-8_W7.62mm, symbol Amplifier_Audio:LM386
