File: select.sch (KiCad schematic (older format))
At the start: 17 parts, among them U201 7402

Commit message: Latch
Parts:
- MX201, MX202, MX203, MX204: footprint MX_Only:MXOnly-1U -> MX_Only:MXOnly-1U-NoLED
- renumbered D205 to D?, D208 to D?, D207 to D?, D206 to D?, D201 to D?, D204 to D?, D203 to D?, D202 to D?
Changed lines of the file:
@@
 $Descr A4 11693 8268
 encoding utf-8
-Sheet 2 4
+Sheet 3 3
 Title "Audio Switch with Amp"
 Date "2021-09-06"
@@
 c
 $Comp
-L Device:D_Small D205
+L Device:D_Small D?
 U 1 1 62DE8D22
 P 3800 4350
-F 0 "D205" H 3800 4143 50  0000 C CNN
+F 0 "D?" H 3800 4143 50  0000 C CNN
 F 1 "D_Small" H 3800 4234 50  0000 C CNN
 F 2 "Diode_SMD:D_0805_2012Metric_Pad1.15x1.40mm_HandSolder" V 3800 4350 50  0001 C CNN
@@
 $EndComp
 $Comp
-L Device:D_Small D208
+L Device:D_Small D?
 U 1 1 62DEABF5
 P 3800 5900
-F 0 "D208" H 3800 5693 50  0000 C CNN
+F 0 "D?" H 3800 5693 50  0000 C CNN
 F 1 "D_Small" H 3800 5784 50  0000 C CNN
 F 2 "Diode_SMD:D_0805_2012Metric_Pad1.15x1.40mm_HandSolder" V 3800 5900 50  0001 C CNN
@@
 $EndComp
 $Comp
-L Device:D_Small D207
+L Device:D_Small D?
 U 1 1 62DEC02A
 P 3800 5550
-F 0 "D207" H 3800 5343 50  0000 C CNN
+F 0 "D?" H 3800 5343 50  0000 C CNN
 F 1 "D_Small" H 3800 5434 50  0000 C CNN
 F 2 "Diode_SMD:D_0805_2012Metric_Pad1.15x1.40mm_HandSolder" V 3800 5550 50  0001 C CNN
@@
 $EndComp
 $Comp
-L Device:D_Small D206
+L Device:D_Small D?
 U 1 1 62DED8FB
 P 3800 4700
-F 0 "D206" H 3800 4493 50  0000 C CNN
+F 0 "D?" H 3800 4493 50  0000 C CNN
 F 1 "D_Small" H 3800 4584 50  0000 C CNN
 F 2 "Diode_SMD:D_0805_2012Metric_Pad1.15x1.40mm_HandSolder" V 3800 4700 50  0001 C CNN
@@
 $EndComp
 $Comp
-L Device:D_Small D201
+L Device:D_Small D?
 U 1 1 62DF2F79
 P 3800 1900
-F 0 "D201" H 3800 1693 50  0000 C CNN
+F 0 "D?" H 3800 1693 50  0000 C CNN
 F 1 "D_Small" H 3800 1784 50  0000 C CNN
 F 2 "Diode_SMD:D_0805_2012Metric_Pad1.15x1.40mm_HandSolder" V 3800 1900 50  0001 C CNN
@@
 $EndComp
 $Comp
-L Device:D_Small D204
+L Device:D_Small D?
 U 1 1 62DF2F7F
 P 3800 3500
-F 0 "D204" H 3800 3293 50  0000 C CNN
+F 0 "D?" H 3800 3293 50  0000 C CNN
 F 1 "D_Small" H 3800 3384 50  0000 C CNN
 F 2 "Diode_SMD:D_0805_2012Metric_Pad1.15x1.40mm_HandSolder" V 3800 3500 50  0001 C CNN
@@
 $EndComp
 $Comp
-L Device:D_Small D203
+L Device:D_Small D?
 U 1 1 62DF2F85
 P 3800 3150
-F 0 "D203" H 3800 2943 50  0000 C CNN
+F 0 "D?" H 3800 2943 50  0000 C CNN
 F 1 "D_Small" H 3800 3034 50  0000 C CNN
 F 2 "Diode_SMD:D_0805_2012Metric_Pad1.15x1.40mm_HandSolder" V 3800 3150 50  0001 C CNN
@@
 $EndComp
 $Comp
-L Device:D_Small D202
+L Device:D_Small D?
 U 1 1 62DF2F8B
 P 3800 2250
-F 0 "D202" H 3800 2043 50  0000 C CNN
+F 0 "D?" H 3800 2043 50  0000 C CNN
 F 1 "D_Small" H 3800 2134 50  0000 C CNN
 F 2 "Diode_SMD:D_0805_2012Metric_Pad1.15x1.40mm_HandSolder" V 3800 2250 50  0001 C CNN
@@
 F 0 "MX204" H 4083 5523 60  0000 C CNN
 F 1 "MX-NoLED" H 4083 5449 20  0000 C CNN
-F 2 "MX_Only:MXOnly-1U" H 3425 5275 60  0001 C CNN
+F 2 "MX_Only:MXOnly-1U-NoLED" H 3425 5275 60  0001 C CNN
 F 3 "" H 3425 5275 60  0001 C CNN
 	1    4050 5300
@@
 F 0 "MX203" H 4083 4323 60  0000 C CNN
 F 1 "MX-NoLED" H 4083 4249 20  0000 C CNN
-F 2 "MX_Only:MXOnly-1U" H 3425 4075 60  0001 C CNN
+F 2 "MX_Only:MXOnly-1U-NoLED" H 3425 4075 60  0001 C CNN
 F 3 "" H 3425 4075 60  0001 C CNN
 	1    4050 4100
@@
 F 0 "MX202" H 4133 3123 60  0000 C CNN
 F 1 "MX-NoLED" H 4133 3049 20  0000 C CNN
-F 2 "MX_Only:MXOnly-1U" H 3475 2875 60  0001 C CNN
+F 2 "MX_Only:MXOnly-1U-NoLED" H 3475 2875 60  0001 C CNN
 F 3 "" H 3475 2875 60  0001 C CNN
 	1    4100 2900
@@
 F 0 "MX201" H 4133 1873 60  0000 C CNN
 F 1 "MX-NoLED" H 4133 1799 20  0000 C CNN
-F 2 "MX_Only:MXOnly-1U" H 3475 1625 60  0001 C CNN
+F 2 "MX_Only:MXOnly-1U-NoLED" H 3475 1625 60  0001 C CNN
 F 3 "" H 3475 1625 60  0001 C CNN
 	1    4100 1650
