File: audio-switch.sch (KiCad schematic (older format))
At the start: 21 parts, among them J1 OUT_1, U1 Pico, U2 CD4052B, U3 CD4052B

Commit message: Remove pico and use sr latch for input slection
Parts:
- removed MX1, MX2, MX3, MX4: MX-LED, MX_Only:MXOnly-1U, symbol MX_Alps_Hybrid:MX-LED
- removed U1: Pico, pi:RPi_Pico_SMD_TH, symbol MCU_RaspberryPi_and_Boards:Pico
- added D5, D6, D7, D8: D_Small, Diode_SMD:D_0805_2012Metric_Pad1.15x1.40mm_HandSolder, symbol Device:D_Small
- added MX1, MX2, MX3, MX4: MX-NoLED, MX_Only:MXOnly-1U, symbol MX_Alps_Hybrid:MX-NoLED
- added U4: 7402, Package_DIP:DIP-14_W7.62mm, symbol 74xx:7402
- OUT_2: value AudioJack4_Out -> OUT_2
- R1, R2, R3, R4: value R_Led -> R_Small
- U2, U3: footprint Package_DIP:DIP-16_W7.62mm_Socket -> Package_DIP:DIP-16_W7.62mm
- renumbered IN_1 to IN_0, IN_4 to IN_1, J1 to OUT_1
Connections:
- net labels added: Select_A_HIGH, Select_A_LOW, Select_B_HIGH, Select_B_LOW
- net labels removed: +3.3V, Col0, Col1, GNDA, LEDCol0, LEDCol1, LEDRow0, LEDRow1, Row0, Row1
- wire segments 165 -> 132
Other:
- moved on the sheet: IN_0, IN_1, IN_2, IN_3, OUT_1, OUT_2, U2, U3

Commit message: Added amps
Parts:
- removed D1, D2, D3, D4, D5, D6, D7, D8: D_Small, Diode_SMD:D_0805_2012Metric_Pad1.15x1.40mm_HandSolder, symbol Device:D_Small
- removed IN_0, IN_1, IN_2, IN_3: AudioJack4_IN, Connector_Audio:Jack_3.5mm_PJ320E_Horizontal, symbol Connector:AudioJack4
- removed MX1, MX2, MX3, MX4: MX-NoLED, MX_Only:MXOnly-1U, symbol MX_Alps_Hybrid:MX-NoLED
- removed R1, R2, R3, R4: R_Small, Resistor_SMD:R_0805_2012Metric_Pad1.20x1.40mm_HandSolder, symbol Device:R_Small
- removed U2, U3: CD4052B, Package_DIP:DIP-16_W7.62mm, symbol Analog_Switch:CD4052B
- removed U4: 7402, Package_DIP:DIP-14_W7.62mm, symbol 74xx:7402
- renumbered OUT_1 to OUT_101, OUT_2 to OUT_102
Connections:
- net Out_R1 renamed Out_Right
- net Out_R2 renamed GNDS
- net Out_S renamed Mic
- net Out_T renamed Out_Left
Other:
- moved on the sheet: OUT_101, OUT_102

Commit message: refactor
Parts:
- added IN_? (x4): AudioJack4_IN, Connector_Audio:Jack_3.5mm_PJ320E_Horizontal, symbol Connector:AudioJack4
- added U? (x2): DG509A, Package_DIP:DIP-16_W7.62mm, symbol 74xx-GEORGE:DG509A
Connections:
- net GNDS: now also U?.8 (A_Ouput)
- net Mic: now also U?.9 (B_Output)
- new net: IN_?.R1, U?.10 (S4B)
- new net: IN_?.R2, U?.7 (S4A)
- new net: IN_?.S, U?.10 (S4B)
- new net: IN_?.T, U?.7 (S4A)
- new net: IN_?.R1, U?.11 (S3B)
- new net: IN_?.R1, U?.12 (S2B)
- new net: IN_?.R1, U?.13 (S1B)
- new net: IN_?.T, U?.4 (S1A)
- new net: IN_?.T, U?.5 (S2A)
- new net: IN_?.T, U?.6 (S3A)
- new net: IN_?.S, U?.11 (S3B)
- new net: IN_?.S, U?.12 (S2B)
- new net: IN_?.S, U?.13 (S1B)
- new net: IN_?.R2, U?.4 (S1A)
- new net: IN_?.R2, U?.5 (S2A)
- new net: IN_?.R2, U?.6 (S3A)
- new net +5V: U?.14 (V+), U?.14 (V+), U?.2 (Enable), U?.2 (Enable)
- new net GND: U?.15 (GND), U?.15 (GND)
- new net Input_Left: U?.8 (A_Ouput)
- new net Input_Right: U?.9 (B_Output)
- new net Select_A: U?.1 (A0), U?.1 (A0)
- new net Select_B: U?.16 (A1), U?.16 (A1)
Other:
- note added: "Audio Out"
- note added: "Audio Switch"
- moved on the sheet: OUT_101, OUT_102

Commit message: Latch
Parts:
- removed IN_? (x4): AudioJack4_IN, Connector_Audio:Jack_3.5mm_PJ320E_Horizontal, symbol Connector:AudioJack4
- removed OUT_101: OUT_1, Connector_Audio:Jack_3.5mm_PJ320E_Horizontal, symbol Connector:AudioJack4
- removed OUT_102: OUT_2, Connector_Audio:Jack_3.5mm_PJ320E_Horizontal, symbol Connector:AudioJack4
- removed U? (x2): DG509A, Package_DIP:DIP-16_W7.62mm, symbol 74xx-GEORGE:DG509A
- added BASS1, GAIN1, VOL1: 10k, Potentiometer_THT:Potentiometer_Alps_RK09L_Double_Vertical, symbol Device:R_POT_Dual_Separate
- added C1, C10, C12, C17, C3, C8: 0.1u, Capacitor_SMD:C_0805_2012Metric_Pad1.18x1.45mm_HandSolder, symbol Device:C_Small
- added C11, C2: 100u, Capacitor_SMD:C_0805_2012Metric_Pad1.18x1.45mm_HandSolder, symbol Device:CP
- added C13, C4: 470p, Capacitor_SMD:C_0805_2012Metric_Pad1.18x1.45mm_HandSolder, symbol Device:C_Small
- added C14, C15, C5, C6: 10u, Capacitor_SMD:C_0805_2012Metric_Pad1.18x1.45mm_HandSolder, symbol Device:CP
- added C16, C7: 0.033u, Capacitor_SMD:C_0805_2012Metric_Pad1.18x1.45mm_HandSolder, symbol Device:C_Small
- added C18, C9: 1000u, Capacitor_SMD:C_0805_2012Metric_Pad1.18x1.45mm_HandSolder, symbol Device:CP
- added D1, D2, D3, D4, D5, D6, D7, D8: D_Small, Diode_SMD:D_0805_2012Metric_Pad1.15x1.40mm_HandSolder, symbol Device:D_Small
- added IN_1, IN_2, IN_3, IN_4: AudioJack4_IN, Connector_Audio:Jack_3.5mm_PJ320E_Horizontal, symbol Connector:AudioJack4
- added MX1, MX2, MX3, MX4: MX-NoLED, MX_Only:MXOnly-1U-NoLED, symbol MX_Alps_Hybrid:MX-NoLED
- added OUT_1: OUT_1, Connector_Audio:Jack_3.5mm_PJ320E_Horizontal, symbol Connector:AudioJack4
- added R1, R2, R3, R4: 10k, Resistor_SMD:R_0805_2012Metric_Pad1.20x1.40mm_HandSolder, symbol Device:R_Small
- added R5, R7: 10k, Resistor_SMD:R_0805_2012Metric_Pad1.20x1.40mm_HandSolder, symbol Device:R
- added R6, R8: 10, Resistor_SMD:R_0805_2012Metric_Pad1.20x1.40mm_HandSolder, symbol Device:R
- added U1: 7402, Package_DIP:DIP-14_W7.62mm, symbol 74xx:7402
- added U2, U3: DG509A, Package_DIP:DIP-16_W7.62mm, symbol 74xx-GEORGE:DG509A
- added U4, U5: LM386, Package_DIP:DIP-8_W7.62mm, symbol Amplifier_Audio:LM386
Connections:
- net +5V: now also C1.1, C10.1, C11.1, C12.2, C2.1, C3.2, MX1.1 (COL), MX2.1 (COL), MX3.1 (COL), MX4.1 (COL), U1.14 (VCC), U2.14 (V+), U2.2 (Enable), U3.14 (V+), U3.2 (Enable), U4.6 (V+), U5.6 (V+)
- net GND: now also C1.2, C10.2, C11.2, C12.1, C13.1, C13.2, C15.2, C2.2, C3.1, C4.1, C4.2, C6.2, R1.2, R2.2, R3.2, R4.2, R6.2, R8.2, U1.7 (GND), U2.15 (GND), U3.15 (GND), U4.2 (-), U4.4 (GND), U5.2 (-), U5.4 (GND), VOL1.3, VOL1.6
- net GNDS: now also OUT_1.R2, U3.8 (A_Ouput)
- net Input_Left: now also U2.8 (A_Ouput), VOL1.4
- net Input_Right: now also U2.9 (B_Output), VOL1.1
- net Out_Left: now also C18.1, OUT_1.T
- net Out_Right: now also C9.1, OUT_1.R1
- net Select_A: now also U1.1, U1.5, U2.1 (A0), U3.1 (A0)
- net Select_B: now also U1.10, U1.11, U2.16 (A1), U3.16 (A1)
- new net: IN_4.R1, U2.10 (S4B)
- new net: IN_4.R2, U3.7 (S4A)
- new net: IN_4.S, U3.10 (S4B)
- new net: IN_4.T, U2.7 (S4A)
- new net: IN_3.R1, U2.11 (S3B)
- new net: IN_2.R1, U2.12 (S2B)
- new net: IN_1.R1, U2.13 (S1B)
- new net: IN_1.T, U2.4 (S1A)
- new net: IN_2.T, U2.5 (S2A)
- new net: IN_3.T, U2.6 (S3A)
- new net: IN_3.S, U3.11 (S3B)
- new net: IN_2.S, U3.12 (S2B)
- new net: IN_1.S, U3.13 (S1B)
- new net: IN_1.R2, U3.4 (S1A)
- new net: IN_2.R2, U3.5 (S2A)
- new net: IN_3.R2, U3.6 (S3A)
- new net: BASS1.5, GAIN1.5, U5.1 (GAIN)
- new net: U5.3 (+), VOL1.5
- new net: C16.2, C17.1, C18.2, U5.5
- new net: R7.1, U5.7 (BYPASS)
- new net: C14.2, U5.8 (GAIN)
- new net: C15.1, R7.2
- new net: C17.2, R8.1
- new net: BASS1.6, C16.1
- new net: C14.1, GAIN1.6
- new net: BASS1.2, GAIN1.2, U4.1 (GAIN)
- new net: U4.3 (+), VOL1.2
- new net: C7.2, C8.1, C9.2, U4.5
- new net: R5.1, U4.7 (BYPASS)
- new net: C5.2, U4.8 (GAIN)
- new net: C6.1, R5.2
- new net: C8.2, R6.1
- new net: BASS1.3, C7.1
- new net: C5.1, GAIN1.3
- new net: D1.2 (A), D2.2 (A), MX3.2 (ROW)
- new net: D3.2 (A), D4.2 (A), MX4.2 (ROW)
- new net: D5.2 (A), D6.2 (A), MX1.2 (ROW)
- new net: D7.2 (A), D8.2 (A), MX2.2 (ROW)
- new net: U1.13, U1.9
- new net: U1.3, U1.4
- new net a: D3.1 (K), D7.1 (K), R1.1, U1.2
- new net b: D1.1 (K), D5.1 (K), R2.1, U1.6
- new net c: D6.1 (K), D8.1 (K), R3.1, U1.8
- new net d: D2.1 (K), D4.1 (K), R4.1, U1.12
- new net mic: OUT_1.S, U3.9 (B_Output)
Other:
- note added: "Amp\n"
- note added: "Power\n"
- note added: "Pull Down\n"
- note added: "Select Button\n"
- note added: "Select Latch\n"

Commit message: Board designed.
Parts:
- added H101, H102, H103, H104: MountingHole_Pad, MountingHole:MountingHole_2.2mm_M2, symbol Mechanical:MountingHole_Pad
- added J101: USB_C_Receptacle, Connector_USB:USB_C_Receptacle_Amphenol_12401610E4-2A, symbol Connector:USB_C_Receptacle
Connections:
- net +5V: now also J101.A4 (VBUS), J101.A9 (VBUS), J101.B4 (VBUS), J101.B9 (VBUS)
- net GND: now also J101.A1 (GND), J101.A12 (GND), J101.B1 (GND), J101.B12 (GND), J101.S1 (SHIELD)
- no-connect marks 0 -> 22
