File: audio-switch.sch (KiCad schematic (older format))
At the start: 5 parts, among them J101 USB_B_Micro

Commit message: Test
Parts:
- J101: footprint (none) -> Connector_USB:USB_Micro-B_Amphenol_10118194_Horizontal
Connections:
- no-connect marks 4 -> 8
Other:
- moved on the sheet: J101
Changed lines of the file:
@@
 F1 "Power.sch" 50
 $EndSheet
+NoConn ~ 3500 1900
+NoConn ~ 3500 2400
+NoConn ~ 4650 2400
+NoConn ~ 4650 1900
+Wire Wire Line
+	5800 7000 5700 7000
+Wire Wire Line
+	5700 7100 5800 7100
+Wire Wire Line
+	5800 7200 5700 7200
+Wire Wire Line
+	5400 7400 5400 7500
+Wire Wire Line
+	5300 7500 5300 7400
+NoConn ~ 5300 7500
+$Comp
+L Connector:USB_B_Micro J101
+U 1 1 61709797
+P 5400 7000
+F 0 "J101" H 5457 7467 50  0000 C CNN
+F 1 "USB_B_Micro" H 5457 7376 50  0000 C CNN
+F 2 "Connector_USB:USB_Micro-B_Amphenol_10118194_Horizontal" H 5550 6950 50  0001 C CNN
+F 3 "~" H 5550 6950 50  0001 C CNN
+	1    5400 7000
+	1    0    0    -1
+$EndComp
+Wire Wire Line
+	5800 6800 5800 6750
+Wire Wire Line
+	5700 6800 5800 6800
+$Comp
+L power:+5V #PWR0102
+U 1 1 617D1198
+P 5800 6750
+AR Path="/617D1198" Ref="#PWR0102"  Part="1"
+AR Path="/626D4311/617D1198" Ref="#PWR?"  Part="1"
+F 0 "#PWR0102" H 5800 6600 50  0001 C CNN
+F 1 "+5V" H 5815 6923 50  0000 C CNN
+F 2 "" H 5800 6750 50  0001 C CNN
+F 3 "" H 5800 6750 50  0001 C CNN
+	1    5800 6750
+	1    0    0    -1
+$EndComp
+NoConn ~ 5800 7100
+NoConn ~ 5800 7000
+NoConn ~ 5800 7200
 $Comp
 L power:GND #PWR0101
 U 1 1 617D117C
-P 3150 6100
-F 0 "#PWR0101" H 3150 5850 50  0001 C CNN
-F 1 "GND" H 3155 5927 50  0000 C CNN
-F 2 "" H 3150 6100 50  0001 C CNN
-F 3 "" H 3150 6100 50  0001 C CNN
-	1    3150 6100
+P 5400 7500
+F 0 "#PWR0101" H 5400 7250 50  0001 C CNN
+F 1 "GND" H 5405 7327 50  0000 C CNN
+F 2 "" H 5400 7500 50  0001 C CNN
+F 3 "" H 5400 7500 50  0001 C CNN
+	1    5400 7500
 	1    0    0    -1
 $EndComp
-NoConn ~ 3550 5800
-NoConn ~ 3550 5600
-NoConn ~ 3550 5700
-$Comp
-L power:+5V #PWR0102
-U 1 1 617D1198
-P 3550 5350
-AR Path="/617D1198" Ref="#PWR0102"  Part="1"
-AR Path="/626D4311/617D1198" Ref="#PWR?"  Part="1"
-F 0 "#PWR0102" H 3550 5200 50  0001 C CNN
-F 1 "+5V" H 3565 5523 50  0000 C CNN
-F 2 "" H 3550 5350 50  0001 C CNN
-F 3 "" H 3550 5350 50  0001 C CNN
-	1    3550 5350
-	1    0    0    -1
-$EndComp
-Wire Wire Line
-	3450 5400 3550 5400
-Wire Wire Line
-	3550 5400 3550 5350
-$Comp
-L Connector:USB_B_Micro J101
-U 1 1 61709797
-P 3150 5600
-F 0 "J101" H 3207 6067 50  0000 C CNN
-F 1 "USB_B_Micro" H 3207 5976 50  0000 C CNN
-F 2 "" H 3300 5550 50  0001 C CNN
-F 3 "~" H 3300 5550 50  0001 C CNN
-	1    3150 5600
-	1    0    0    -1
-$EndComp
-NoConn ~ 3050 6100
-Wire Wire Line
-	3050 6100 3050 6000
-Wire Wire Line
-	3150 6000 3150 6100
-Wire Wire Line
-	3550 5800 3450 5800
-Wire Wire Line
-	3450 5700 3550 5700
-Wire Wire Line
-	3550 5600 3450 5600
 $EndSCHEMATC
