File: Power.sch (KiCad schematic (older format))
At the start: 12 parts, among them Q501 IRLZ44N, U501 ATtiny85-20PU

Commit message: Test
Parts:
- C501, C502: footprint (none) -> Capacitor_Tantalum_SMD:CP_EIA-2012-15_AVX-P_Pad1.30x1.05mm_HandSolder
- D501: footprint (none) -> Diode_THT:D_DO-41_SOD81_P7.62mm_Horizontal
- L501: footprint (none) -> Inductor_THT:L_Radial_D6.0mm_P4.00mm
- R501, R502, R503, R504, R505: footprint (none) -> Resistor_SMD:R_0805_2012Metric_Pad1.20x1.40mm_HandSolder
- RV501: footprint (none) -> audio-switch:pot_jaycar
Connections:
- no-connect marks 0 -> 3
Changed lines of the file:
@@
 F 0 "C501" H 2688 3296 50  0000 L CNN
 F 1 "47µF" H 2688 3205 50  0000 L CNN
-F 2 "" H 2600 3250 50  0001 C CNN
+F 2 "Capacitor_Tantalum_SMD:CP_EIA-2012-15_AVX-P_Pad1.30x1.05mm_HandSolder" H 2600 3250 50  0001 C CNN
 F 3 "~" H 2600 3250 50  0001 C CNN
 	1    2600 3250
@@
 F 0 "L501" H 5950 2465 50  0000 C CNN
 F 1 "100µH" H 5950 2374 50  0000 C CNN
-F 2 "" H 5950 2250 50  0001 C CNN
+F 2 "Inductor_THT:L_Radial_D6.0mm_P4.00mm" H 5950 2250 50  0001 C CNN
 F 3 "~" H 5950 2250 50  0001 C CNN
 	1    5950 2250
@@
 F 0 "D501" H 6900 2033 50  0000 C CNN
 F 1 "1N5819" H 6900 2124 50  0000 C CNN
-F 2 "" H 6900 2250 50  0001 C CNN
+F 2 "Diode_THT:D_DO-41_SOD81_P7.62mm_Horizontal" H 6900 2250 50  0001 C CNN
 F 3 "~" H 6900 2250 50  0001 C CNN
 	1    6900 2250
@@
 F 0 "C502" H 7338 3046 50  0000 L CNN
 F 1 "47µF" H 7338 2955 50  0000 L CNN
-F 2 "" H 7250 3000 50  0001 C CNN
+F 2 "Capacitor_Tantalum_SMD:CP_EIA-2012-15_AVX-P_Pad1.30x1.05mm_HandSolder" H 7250 3000 50  0001 C CNN
 F 3 "~" H 7250 3000 50  0001 C CNN
 	1    7250 3000
@@
 F 0 "R501" H 5870 3046 50  0000 L CNN
 F 1 "100Ω" H 5870 2955 50  0000 L CNN
-F 2 "" V 5730 3000 50  0001 C CNN
+F 2 "Resistor_SMD:R_0805_2012Metric_Pad1.20x1.40mm_HandSolder" V 5730 3000 50  0001 C CNN
 F 3 "~" H 5800 3000 50  0001 C CNN
 	1    5800 3000
@@
 F 0 "R503" H 8470 2596 50  0000 L CNN
 F 1 "10kΩ" H 8470 2505 50  0000 L CNN
-F 2 "" V 8330 2550 50  0001 C CNN
+F 2 "Resistor_SMD:R_0805_2012Metric_Pad1.20x1.40mm_HandSolder" V 8330 2550 50  0001 C CNN
 F 3 "~" H 8400 2550 50  0001 C CNN
 	1    8400 2550
@@
 F 0 "R504" H 8470 2996 50  0000 L CNN
 F 1 "1kΩ" H 8470 2905 50  0000 L CNN
-F 2 "" V 8330 2950 50  0001 C CNN
+F 2 "Resistor_SMD:R_0805_2012Metric_Pad1.20x1.40mm_HandSolder" V 8330 2950 50  0001 C CNN
 F 3 "~" H 8400 2950 50  0001 C CNN
 	1    8400 2950
@@
 F 0 "R505" H 8470 3496 50  0000 L CNN
 F 1 "2kΩ" H 8470 3405 50  0000 L CNN
-F 2 "" V 8330 3450 50  0001 C CNN
+F 2 "Resistor_SMD:R_0805_2012Metric_Pad1.20x1.40mm_HandSolder" V 8330 3450 50  0001 C CNN
 F 3 "~" H 8400 3450 50  0001 C CNN
 	1    8400 3450
@@
 F 0 "RV501" H 5280 3254 50  0000 R CNN
 F 1 "100kΩ" H 5280 3345 50  0000 R CNN
-F 2 "" H 5350 3300 50  0001 C CNN
+F 2 "audio-switch:pot_jaycar" H 5350 3300 50  0001 C CNN
 F 3 "~" H 5350 3300 50  0001 C CNN
 	1    5350 3300
@@
 F 0 "R502" H 6080 3204 50  0000 R CNN
 F 1 "10kΩ" H 6080 3295 50  0000 R CNN
-F 2 "" V 6080 3250 50  0001 C CNN
+F 2 "Resistor_SMD:R_0805_2012Metric_Pad1.20x1.40mm_HandSolder" V 6080 3250 50  0001 C CNN
 F 3 "~" H 6150 3250 50  0001 C CNN
 	1    6150 3250
@@
 Wire Wire Line
 	5950 3000 6150 3000
+NoConn ~ 4750 2900
+NoConn ~ 4750 3100
+NoConn ~ 4750 3400
 $EndSCHEMATC
