File: Select.sch (KiCad schematic (older format))
At the start: 17 parts, among them U301 7402

Commit message: Test
Parts:
- D301, D302, D303, D304, D305, D306, D307, D308: footprint (none) -> Diode_SMD:D_0805_2012Metric_Pad1.15x1.40mm_HandSolder
- R301, R302, R303, R304: footprint (none) -> Resistor_SMD:R_0805_2012Metric_Pad1.20x1.40mm_HandSolder
Changed lines of the file:
@@
 F 0 "D302" H 2800 2143 50  0000 C CNN
 F 1 "D_Small" H 2800 2234 50  0000 C CNN
-F 2 "" V 2800 2350 50  0001 C CNN
+F 2 "Diode_SMD:D_0805_2012Metric_Pad1.15x1.40mm_HandSolder" V 2800 2350 50  0001 C CNN
 F 3 "~" V 2800 2350 50  0001 C CNN
 	1    2800 2350
@@
 F 0 "D303" H 2800 3043 50  0000 C CNN
 F 1 "D_Small" H 2800 3134 50  0000 C CNN
-F 2 "" V 2800 3250 50  0001 C CNN
+F 2 "Diode_SMD:D_0805_2012Metric_Pad1.15x1.40mm_HandSolder" V 2800 3250 50  0001 C CNN
 F 3 "~" V 2800 3250 50  0001 C CNN
 	1    2800 3250
@@
 F 0 "D304" H 2800 3393 50  0000 C CNN
 F 1 "D_Small" H 2800 3484 50  0000 C CNN
-F 2 "" V 2800 3600 50  0001 C CNN
+F 2 "Diode_SMD:D_0805_2012Metric_Pad1.15x1.40mm_HandSolder" V 2800 3600 50  0001 C CNN
 F 3 "~" V 2800 3600 50  0001 C CNN
 	1    2800 3600
@@
 F 0 "D301" H 2800 1793 50  0000 C CNN
 F 1 "D_Small" H 2800 1884 50  0000 C CNN
-F 2 "" V 2800 2000 50  0001 C CNN
+F 2 "Diode_SMD:D_0805_2012Metric_Pad1.15x1.40mm_HandSolder" V 2800 2000 50  0001 C CNN
 F 3 "~" V 2800 2000 50  0001 C CNN
 	1    2800 2000
@@
 F 0 "D306" H 2800 4593 50  0000 C CNN
 F 1 "D_Small" H 2800 4684 50  0000 C CNN
-F 2 "" V 2800 4800 50  0001 C CNN
+F 2 "Diode_SMD:D_0805_2012Metric_Pad1.15x1.40mm_HandSolder" V 2800 4800 50  0001 C CNN
 F 3 "~" V 2800 4800 50  0001 C CNN
 	1    2800 4800
@@
 F 0 "D307" H 2800 5443 50  0000 C CNN
 F 1 "D_Small" H 2800 5534 50  0000 C CNN
-F 2 "" V 2800 5650 50  0001 C CNN
+F 2 "Diode_SMD:D_0805_2012Metric_Pad1.15x1.40mm_HandSolder" V 2800 5650 50  0001 C CNN
 F 3 "~" V 2800 5650 50  0001 C CNN
 	1    2800 5650
@@
 F 0 "D308" H 2800 5793 50  0000 C CNN
 F 1 "D_Small" H 2800 5884 50  0000 C CNN
-F 2 "" V 2800 6000 50  0001 C CNN
+F 2 "Diode_SMD:D_0805_2012Metric_Pad1.15x1.40mm_HandSolder" V 2800 6000 50  0001 C CNN
 F 3 "~" V 2800 6000 50  0001 C CNN
 	1    2800 6000
@@
 F 0 "D305" H 2800 4243 50  0000 C CNN
 F 1 "D_Small" H 2800 4334 50  0000 C CNN
-F 2 "" V 2800 4450 50  0001 C CNN
+F 2 "Diode_SMD:D_0805_2012Metric_Pad1.15x1.40mm_HandSolder" V 2800 4450 50  0001 C CNN
 F 3 "~" V 2800 4450 50  0001 C CNN
 	1    2800 4450
@@
 F 0 "R304" H 6009 5596 50  0000 L CNN
 F 1 "10kΩ" H 6009 5505 50  0000 L CNN
-F 2 "" H 5950 5550 50  0001 C CNN
+F 2 "Resistor_SMD:R_0805_2012Metric_Pad1.20x1.40mm_HandSolder" H 5950 5550 50  0001 C CNN
 F 3 "~" H 5950 5550 50  0001 C CNN
 	1    5950 5550
@@
 F 0 "R302" H 5109 5596 50  0000 L CNN
 F 1 "10kΩ" H 5109 5505 50  0000 L CNN
-F 2 "" H 5050 5550 50  0001 C CNN
+F 2 "Resistor_SMD:R_0805_2012Metric_Pad1.20x1.40mm_HandSolder" H 5050 5550 50  0001 C CNN
 F 3 "~" H 5050 5550 50  0001 C CNN
 	1    5050 5550
@@
 F 0 "R301" H 4659 5596 50  0000 L CNN
 F 1 "10kΩ" H 4659 5505 50  0000 L CNN
-F 2 "" H 4600 5550 50  0001 C CNN
+F 2 "Resistor_SMD:R_0805_2012Metric_Pad1.20x1.40mm_HandSolder" H 4600 5550 50  0001 C CNN
 F 3 "~" H 4600 5550 50  0001 C CNN
 	1    4600 5550
@@
 F 0 "R303" H 5559 5596 50  0000 L CNN
 F 1 "10kΩ" H 5559 5505 50  0000 L CNN
-F 2 "" H 5500 5550 50  0001 C CNN
+F 2 "Resistor_SMD:R_0805_2012Metric_Pad1.20x1.40mm_HandSolder" H 5500 5550 50  0001 C CNN
 F 3 "~" H 5500 5550 50  0001 C CNN
 	1    5500 5550
