File: audio-switch.kicad_pcb (KiCad board)
At the start: 2 copper layers, 99.5 x 58 mm, 56 parts, among them J101 USB_C_Receptacle, U1 7402, U2 DG509A, U3 DG509A, U4 LM386, U5 LM386

Commit message: Test
Parts:
- removed BASS1, GAIN1, VOL1: 10k, Potentiometer_THT:Potentiometer_Alps_RK09L_Double_Vertical
- removed C1, C10, C12, C17, C3, C8: 0.1u, Capacitor_SMD:C_0805_2012Metric_Pad1.18x1.45mm_HandSolder
- removed C11, C2: 100u, Capacitor_SMD:C_0805_2012Metric_Pad1.18x1.45mm_HandSolder
- removed C13, C4: 470p, Capacitor_SMD:C_0805_2012Metric_Pad1.18x1.45mm_HandSolder
- removed C14, C15, C5, C6: 10u, Capacitor_SMD:C_0805_2012Metric_Pad1.18x1.45mm_HandSolder
- removed C16, C7: 0.033u, Capacitor_SMD:C_0805_2012Metric_Pad1.18x1.45mm_HandSolder
- removed C18, C9: 1000u, Capacitor_SMD:C_0805_2012Metric_Pad1.18x1.45mm_HandSolder
- removed D1, D2, D3, D4, D5, D6, D7, D8: D_Small, Diode_SMD:D_0805_2012Metric_Pad1.15x1.40mm_HandSolder
- removed IN_1, IN_2, IN_3, IN_4: AudioJack4_IN, Connector_Audio:Jack_3.5mm_PJ320E_Horizontal
- removed MX1, MX2, MX3, MX4: MX-NoLED, MX_Only:MXOnly-1U-NoLED
- removed OUT_1: OUT_1, Connector_Audio:Jack_3.5mm_PJ320E_Horizontal
- removed R1, R2, R3, R4, R5, R7: 10k, Resistor_SMD:R_0805_2012Metric_Pad1.20x1.40mm_HandSolder
- removed R6, R8: 10, Resistor_SMD:R_0805_2012Metric_Pad1.20x1.40mm_HandSolder
- removed U1: 7402, Package_DIP:DIP-14_W7.62mm
- removed U2, U3: DG509A, Package_DIP:DIP-16_W7.62mm
- removed U4, U5: LM386, Package_DIP:DIP-8_W7.62mm
- added BASS401: 10kΩ, audio-switch:dual_pot_jaycar, F.Cu at (117.5, 127.5)
- added C401: 0.1µF, Capacitor_SMD:C_0805_2012Metric_Pad1.18x1.45mm_HandSolder, F.Cu at (236.0, 161.0)
- added C402: 100µF, Capacitor_SMD:C_0805_2012Metric_Pad1.18x1.45mm_HandSolder, F.Cu at (240.5, 190.5)
- added C403: 0.1µF, Capacitor_SMD:C_0805_2012Metric_Pad1.18x1.45mm_HandSolder, F.Cu at (246.9, 167.0)
- added C404: 470pF, Capacitor_SMD:C_0805_2012Metric_Pad1.18x1.45mm_HandSolder, F.Cu at (240.5, 193.5)
- added C405: 10µF, Capacitor_SMD:C_0805_2012Metric_Pad1.18x1.45mm_HandSolder, F.Cu at (245.3, 190.5)
- added C406: 10µF, Capacitor_SMD:C_0805_2012Metric_Pad1.18x1.45mm_HandSolder, F.Cu at (240.5, 196.5)
- added C407: 0.033µF, Capacitor_SMD:C_0805_2012Metric_Pad1.18x1.45mm_HandSolder, F.Cu at (245.3, 193.5)
- added C408: 0.1µF, Capacitor_SMD:C_0805_2012Metric_Pad1.18x1.45mm_HandSolder, F.Cu at (250.1, 190.5)
- added C409: 1000µF, Capacitor_SMD:C_0805_2012Metric_Pad1.18x1.45mm_HandSolder, F.Cu at (240.5, 199.5)
- added C410: 0.1µF, Capacitor_SMD:C_0805_2012Metric_Pad1.18x1.45mm_HandSolder, F.Cu at (261.3, 167.0)
- added C411: 100µF, Capacitor_SMD:C_0805_2012Metric_Pad1.18x1.45mm_HandSolder, F.Cu at (245.3, 196.5)
- added C412: 0.1µF, Capacitor_SMD:C_0805_2012Metric_Pad1.18x1.45mm_HandSolder, F.Cu at (250.1, 193.5)
- added C413: 470pF, Capacitor_SMD:C_0805_2012Metric_Pad1.18x1.45mm_HandSolder, F.Cu at (254.9, 190.5)
- added C414: 10µF, Capacitor_SMD:C_0805_2012Metric_Pad1.18x1.45mm_HandSolder, F.Cu at (245.3, 199.5)
- added C415: 10µF, Capacitor_SMD:C_0805_2012Metric_Pad1.18x1.45mm_HandSolder, F.Cu at (250.1, 196.5)
- added C416: 0.033µF, Capacitor_SMD:C_0805_2012Metric_Pad1.18x1.45mm_HandSolder, F.Cu at (254.9, 193.5)
- added C417: 0.1µF, Capacitor_SMD:C_0805_2012Metric_Pad1.18x1.45mm_HandSolder, F.Cu at (250.1, 199.5)
- added C501: 47µF, Capacitor_Tantalum_SMD:CP_EIA-2012-15_AVX-P_Pad1.30x1.05mm_HandSolder, F.Cu at (240.5, 206.3)
- added C502: 47µF, Capacitor_Tantalum_SMD:CP_EIA-2012-15_AVX-P_Pad1.30x1.05mm_HandSolder, F.Cu at (240.5, 209.1)
- added D301: D_Small, Diode_SMD:D_0805_2012Metric_Pad1.15x1.40mm_HandSolder, F.Cu at (266.5, 190.5)
- added D302: D_Small, Diode_SMD:D_0805_2012Metric_Pad1.15x1.40mm_HandSolder, F.Cu at (266.5, 193.6)
- added D303: D_Small, Diode_SMD:D_0805_2012Metric_Pad1.15x1.40mm_HandSolder, F.Cu at (271.3, 190.5)
- added D304: D_Small, Diode_SMD:D_0805_2012Metric_Pad1.15x1.40mm_HandSolder, F.Cu at (266.5, 196.6)
- added D305: D_Small, Diode_SMD:D_0805_2012Metric_Pad1.15x1.40mm_HandSolder, F.Cu at (271.3, 193.6)
- added D306: D_Small, Diode_SMD:D_0805_2012Metric_Pad1.15x1.40mm_HandSolder, F.Cu at (276.1, 190.5)
- added D307: D_Small, Diode_SMD:D_0805_2012Metric_Pad1.15x1.40mm_HandSolder, F.Cu at (271.3, 196.6)
- added D308: D_Small, Diode_SMD:D_0805_2012Metric_Pad1.15x1.40mm_HandSolder, F.Cu at (276.1, 193.6)
- added D501: 1N5819, Diode_THT:D_DO-41_SOD81_P7.62mm_Horizontal, F.Cu at (202.0, 127.5)
- added GAIN401: 10kΩ, audio-switch:dual_pot_jaycar, F.Cu at (121.5, 143.5)
- added L501: 100µH, Inductor_THT:L_Radial_D6.0mm_P4.00mm, F.Cu at (211.5, 149.0)
- added MX301: MX-NoLED, MX_Only:MXOnly-1U-NoLED, F.Cu at (137.3, 59.8)
- added MX302: MX-NoLED, MX_Only:MXOnly-1U-NoLED, F.Cu at (137.3, 80.0)
- added MX303: MX-NoLED, MX_Only:MXOnly-1U-NoLED, F.Cu at (157.5, 59.8)
- added MX304: MX-NoLED, MX_Only:MXOnly-1U-NoLED, F.Cu at (157.5, 80.0)
- added Q501: IRLZ44N, Package_TO_SOT_THT:TO-220-3_Vertical, F.Cu at (177.3, 112.8)
- added R301: 10kΩ, Resistor_SMD:R_0805_2012Metric_Pad1.20x1.40mm_HandSolder, F.Cu at (226.6, 111.0)
- added R302: 10kΩ, Resistor_SMD:R_0805_2012Metric_Pad1.20x1.40mm_HandSolder, F.Cu at (235.5, 134.2)
- added R303: 10kΩ, Resistor_SMD:R_0805_2012Metric_Pad1.20x1.40mm_HandSolder, F.Cu at (223.4, 115.7)
- added R304: 10kΩ, Resistor_SMD:R_0805_2012Metric_Pad1.20x1.40mm_HandSolder, F.Cu at (250.5, 115.0)
- added R401: 10kΩ, Resistor_SMD:R_0805_2012Metric_Pad1.20x1.40mm_HandSolder, F.Cu at (223.2, 101.5)
- added R402: 10Ω, Resistor_SMD:R_0805_2012Metric_Pad1.20x1.40mm_HandSolder, F.Cu at (234.8, 128.9)
- added R403: 10kΩ, Resistor_SMD:R_0805_2012Metric_Pad1.20x1.40mm_HandSolder, F.Cu at (223.2, 104.6)
- added R404: 10Ω, Resistor_SMD:R_0805_2012Metric_Pad1.20x1.40mm_HandSolder, F.Cu at (233.8, 101.5)
- added R501: 100Ω, Resistor_SMD:R_0805_2012Metric_Pad1.20x1.40mm_HandSolder, F.Cu at (239.3, 106.9)
- added R502: 10kΩ, Resistor_SMD:R_0805_2012Metric_Pad1.20x1.40mm_HandSolder, F.Cu at (234.8, 117.7)
- added R503: 10kΩ, Resistor_SMD:R_0805_2012Metric_Pad1.20x1.40mm_HandSolder, F.Cu at (239.3, 110.1)
- added R504: 1kΩ, Resistor_SMD:R_0805_2012Metric_Pad1.20x1.40mm_HandSolder, F.Cu at (234.8, 120.9)
- added R505: 2kΩ, Resistor_SMD:R_0805_2012Metric_Pad1.20x1.40mm_HandSolder, F.Cu at (237.2, 124.0)
- added RV501: 100kΩ, audio-switch:pot_jaycar, F.Cu at (188.1, 102.5)
- added U201: DG509A, Package_DIP:DIP-16_W7.62mm, F.Cu at (221.5, 51.8)
- added U202: DG509A, Package_DIP:DIP-16_W7.62mm, F.Cu at (210.7, 51.8)
- added U301: 7402, Package_DIP:DIP-14_W7.62mm, F.Cu at (181.5, 39.5)
- added U401: LM386, Package_DIP:DIP-8_W7.62mm, F.Cu at (93.3, 145.5)
- added U402: LM386, Package_DIP:DIP-8_W7.62mm, F.Cu at (93.3, 157.3)
- added U501: ATtiny85-20PU, Package_DIP:DIP-8_W7.62mm, F.Cu at (175.7, 99.2)
- added VOL401: 10kΩ, audio-switch:dual_pot_jaycar, F.Cu at (101.5, 124.0)
- J101: value USB_C_Receptacle -> USB_B_Micro; footprint Connector_USB:USB_C_Receptacle_Amphenol_12401610E4-2A -> Connector_USB:USB_Micro-B_Amphenol_10118194_Horizontal
- moved H103 139.1 mm to (218.0, 79.6)
- moved H101 133.1 mm to (212.0, 79.6)
- moved J101 65.5 mm to (207.5, 118.0), turned to 0 degrees
- moved H104 52.8 mm to (218.0, 85.6)
- moved H102 41.7 mm to (212.0, 85.6)
Routing:
- net +5V: track 303.9 -> 0.00 mm, vias 3 -> 0
- net Net-(IN_1-PadR2): track 73.7 -> 0.00 mm, vias 2 -> 0
- net Net-(IN_1-PadS): track 65.5 -> 0.00 mm, vias 2 -> 0
- net Input_Right: track 62.4 -> 0.00 mm
- net Net-(IN_2-PadR2): track 59.1 -> 0.00 mm, vias 1 -> 0
- net GND: track 58.8 -> 0.00 mm, vias 14 -> 0
- net Net-(C16-Pad2): track 57.9 -> 0.00 mm, vias 2 -> 0
- net Net-(D1-Pad2): track 57.2 -> 0.00 mm, vias 2 -> 0
- net Net-(IN_1-PadR1): track 53.5 -> 0.00 mm
- net Net-(IN_2-PadS): track 53.1 -> 0.00 mm, vias 1 -> 0
- net Input_Left: track 49.5 -> 0.00 mm
- net Net-(D5-Pad2): track 48.1 -> 0.00 mm, vias 2 -> 0
- net Net-(IN_2-PadR1): track 45.0 -> 0.00 mm
- net Net-(IN_3-PadR2): track 44.7 -> 0.00 mm
- net Net-(IN_3-PadS): track 41.9 -> 0.00 mm
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- removed copper zone on B.Cu, net GND
- removed copper zone on F.Cu, net GND
Other:
- board outline removed
